File: pcb/Swarm-B/Swarm-B.sch (KiCad schematic (older format))
At the start: 25 parts, among them J1 RX_Break, J2 5v_3Pi, J3 GND_3Pi, J4 I2C_3Pi, SW1 Bttn, U1 74LS32, U2 TSDP34138

Commit message: update
Parts:
- R1, R2, R3, R4, R6: footprint Resistor_THT:R_Axial_DIN0204_L3.6mm_D1.6mm_P5.08mm_Horizontal -> Resistor_THT:R_Axial_DIN0204_L3.6mm_D1.6mm_P7.62mm_Horizontal
- U1: footprint Package_DIP:DIP-16_W7.62mm_Socket -> Package_DIP:DIP-14_W7.62mm_Socket
Changed lines of the file:
@@
 F 0 "U1" H 3050 3975 50  0000 C CNN
 F 1 "74LS32" H 3050 3884 50  0000 C CNN
-F 2 "Package_DIP:DIP-16_W7.62mm_Socket" H 3050 3650 50  0001 C CNN
+F 2 "Package_DIP:DIP-14_W7.62mm_Socket" H 3050 3650 50  0001 C CNN
 F 3 "http://www.ti.com/lit/gpn/sn74LS32" H 3050 3650 50  0001 C CNN
 	1    3050 3650
@@
 F 0 "U1" H 3050 4525 50  0000 C CNN
 F 1 "74LS32" H 3050 4434 50  0000 C CNN
-F 2 "Package_DIP:DIP-16_W7.62mm_Socket" H 3050 4200 50  0001 C CNN
+F 2 "Package_DIP:DIP-14_W7.62mm_Socket" H 3050 4200 50  0001 C CNN
 F 3 "http://www.ti.com/lit/gpn/sn74LS32" H 3050 4200 50  0001 C CNN
 	2    3050 4200
@@
 F 0 "U1" H 3050 5075 50  0000 C CNN
 F 1 "74LS32" H 3050 4984 50  0000 C CNN
-F 2 "Package_DIP:DIP-16_W7.62mm_Socket" H 3050 4750 50  0001 C CNN
+F 2 "Package_DIP:DIP-14_W7.62mm_Socket" H 3050 4750 50  0001 C CNN
 F 3 "http://www.ti.com/lit/gpn/sn74LS32" H 3050 4750 50  0001 C CNN
 	3    3050 4750
@@
 F 0 "U1" H 3050 5625 50  0000 C CNN
 F 1 "74LS32" H 3050 5534 50  0000 C CNN
-F 2 "Package_DIP:DIP-16_W7.62mm_Socket" H 3050 5300 50  0001 C CNN
+F 2 "Package_DIP:DIP-14_W7.62mm_Socket" H 3050 5300 50  0001 C CNN
 F 3 "http://www.ti.com/lit/gpn/sn74LS32" H 3050 5300 50  0001 C CNN
 	4    3050 5300
@@
 F 0 "U1" H 3230 2096 50  0000 L CNN
 F 1 "74LS32" H 3230 2005 50  0000 L CNN
-F 2 "Package_DIP:DIP-16_W7.62mm_Socket" H 3000 2050 50  0001 C CNN
+F 2 "Package_DIP:DIP-14_W7.62mm_Socket" H 3000 2050 50  0001 C CNN
 F 3 "http://www.ti.com/lit/gpn/sn74LS32" H 3000 2050 50  0001 C CNN
 	5    3000 2050
@@
 F 0 "R1" V 1605 2618 45  0000 L CNN
 F 1 "15R_IRLED" V 1689 2618 45  0000 L CNN
-F 2 "Resistor_THT:R_Axial_DIN0204_L3.6mm_D1.6mm_P5.08mm_Horizontal" H 1700 2700 20  0001 C CNN
+F 2 "Resistor_THT:R_Axial_DIN0204_L3.6mm_D1.6mm_P7.62mm_Horizontal" H 1700 2700 20  0001 C CNN
 F 3 "" H 1700 2550 60  0001 C CNN
 F 4 " " V 1784 2618 60  0000 L CNN "Field4"
@@
 F 0 "R6" H 7300 3400 45  0000 C CNN
 F 1 "10K_LDR" H 7300 3316 45  0000 C CNN
-F 2 "Resistor_THT:R_Axial_DIN0204_L3.6mm_D1.6mm_P5.08mm_Horizontal" H 7300 3250 20  0001 C CNN
+F 2 "Resistor_THT:R_Axial_DIN0204_L3.6mm_D1.6mm_P7.62mm_Horizontal" H 7300 3250 20  0001 C CNN
 F 3 "" H 7300 3100 60  0001 C CNN
 F 4 " " H 7300 3221 60  0000 C CNN "Field4"
@@
 F 0 "R2" H 4600 4850 45  0000 C CNN
 F 1 "155R_R" H 4600 4766 45  0000 C CNN
-F 2 "Resistor_THT:R_Axial_DIN0204_L3.6mm_D1.6mm_P5.08mm_Horizontal" H 4600 4700 20  0001 C CNN
+F 2 "Resistor_THT:R_Axial_DIN0204_L3.6mm_D1.6mm_P7.62mm_Horizontal" H 4600 4700 20  0001 C CNN
 F 3 "" H 4600 4550 60  0001 C CNN
 F 4 " " H 4600 4671 60  0000 C CNN "Field4"
@@
 F 0 "R3" H 5000 4750 45  0000 C CNN
 F 1 "90R_G" H 5000 4666 45  0000 C CNN
-F 2 "Resistor_THT:R_Axial_DIN0204_L3.6mm_D1.6mm_P5.08mm_Horizontal" H 5000 4600 20  0001 C CNN
+F 2 "Resistor_THT:R_Axial_DIN0204_L3.6mm_D1.6mm_P7.62mm_Horizontal" H 5000 4600 20  0001 C CNN
 F 3 "" H 5000 4450 60  0001 C CNN
 F 4 " " H 5000 4571 60  0000 C CNN "Field4"
@@
 F 0 "R4" H 5400 4650 45  0000 C CNN
 F 1 "85R_B" H 5400 4566 45  0000 C CNN
-F 2 "Resistor_THT:R_Axial_DIN0204_L3.6mm_D1.6mm_P5.08mm_Horizontal" H 5400 4500 20  0001 C CNN
+F 2 "Resistor_THT:R_Axial_DIN0204_L3.6mm_D1.6mm_P7.62mm_Horizontal" H 5400 4500 20  0001 C CNN
 F 3 "" H 5400 4350 60  0001 C CNN
 F 4 " " H 5400 4471 60  0000 C CNN "Field4"

Commit message: altered pcb to house ICs on the underside
Parts:
- VR1, VR2, VR3: footprint Potentiometer_THT:Potentiometer_Bourns_3299P_Horizontal -> Potentiometer_THT:Potentiometer_Bourns_3386F_Vertical
- VR4: footprint Potentiometer_THT:Potentiometer_Bourns_3299P_Horizontal -> Potentiometer_THT:Potentiometer_Bourns_3386P_Vertical
Changed lines of the file:
@@
 F 0 "VR1" H 9083 3945 45  0000 R CNN
 F 1 "10K_Pot_B" H 9083 3861 45  0000 R CNN
-F 2 "Potentiometer_THT:Potentiometer_Bourns_3299P_Horizontal" V 9000 3850 20  0001 C CNN
+F 2 "Potentiometer_THT:Potentiometer_Bourns_3386F_Vertical" V 9000 3850 20  0001 C CNN
 F 3 "" H 9150 3850 60  0001 C CNN
 F 4 "RES-09730" H 9083 3766 60  0000 R CNN "Field4"
@@
 F 0 "VR3" H 9683 3945 45  0000 R CNN
 F 1 "10K_Pot_C" H 9683 3861 45  0000 R CNN
-F 2 "Potentiometer_THT:Potentiometer_Bourns_3299P_Horizontal" V 9600 3850 20  0001 C CNN
+F 2 "Potentiometer_THT:Potentiometer_Bourns_3386F_Vertical" V 9600 3850 20  0001 C CNN
 F 3 "" H 9750 3850 60  0001 C CNN
 F 4 "RES-09730" H 9683 3766 60  0000 R CNN "Field4"
@@
 F 0 "VR2" H 8483 3945 45  0000 R CNN
 F 1 "10K_Pot_A" H 8483 3861 45  0000 R CNN
-F 2 "Potentiometer_THT:Potentiometer_Bourns_3299P_Horizontal" V 8400 3850 20  0001 C CNN
+F 2 "Potentiometer_THT:Potentiometer_Bourns_3386F_Vertical" V 8400 3850 20  0001 C CNN
 F 3 "" H 8550 3850 60  0001 C CNN
 F 4 "RES-09730" H 8483 3766 60  0000 R CNN "Field4"
@@
 F 0 "VR4" H 1833 3245 45  0000 R CNN
 F 1 "1K_Pot_IRLED" H 1833 3161 45  0000 R CNN
-F 2 "Potentiometer_THT:Potentiometer_Bourns_3299P_Horizontal" V 1750 3150 20  0001 C CNN
+F 2 "Potentiometer_THT:Potentiometer_Bourns_3386P_Vertical" V 1750 3150 20  0001 C CNN
 F 3 "" H 1900 3150 60  0001 C CNN
 F 4 "RES-09730" H 1833 3066 60  0000 R CNN "Field4"
